Commit message: modified CameraDepth_sensor_fixedjoint z value

File: share/urdf/pepper.urdf (robot description, URDF)
Before this commit: robot JulietteY20MP, 84 links, 83 joints
Joints:
- joint CameraDepth_sensor_fixedjoint: origin xyz=0.05138 0.039 0.1194 rpy=0 0 0 -> xyz=0.05138 0.039 0.2374 rpy=0 0 0
